Commit message: reconstruction

File: motoman_description/robots/sia5/sia5_with_dhand_and_multi_kinect.urdf.xacro (robot description, xacro)
@@ -6,21 +6,21 @@
   <xacro:include filename="$(find motoman_description)/robots/sia5/sia5_with_dhand.urdf.xacro"/>
   <!-- add Kinect V2 -->
-  <!-- Kinect_second -->
+  <!-- Kinect_center -->
   <!-- Link -->
-  <xacro:kinect2_link_box_v0 name="kinect_second_link"/>
-  <link name="kinect_second_rgb_optical_frame"/>
+  <xacro:kinect2_link_box_v0 name="kinect_center_link"/>
+  <link name="kinect_center_rgb_optical_frame"/>
   <!-- Joint -->
-  <joint name="joint_kinect_second" type="fixed">
-	<origin xyz="1.4828 0.0827 0.3932" rpy="-0.0031 0.4431 3.14" />
+  <joint name="joint_kinect_center" type="fixed">
+	<origin xyz="1.4721 0.0827 0.3932" rpy="-0.0031 0.4431 3.14" />
     <parent link="base_link"/>
-    <child link="kinect_second_link"/>
+    <child link="kinect_center_link"/>
   </joint>
-  <joint name="joint_rgb_kinect_second" type="fixed">
+  <joint name="joint_rgb_kinect_center" type="fixed">
     <origin rpy="${M_PI/2} ${M_PI} ${M_PI/2}"/>
-    <parent link="kinect_second_link"/>
-    <child link="kinect_second_rgb_optical_frame"/>
+    <parent link="kinect_center_link"/>
+    <child link="kinect_center_rgb_optical_frame"/>
   </joint>
   <!-- Gazebo -->
-  <xacro:kinect_gazebo name="kinect_second"/>
+  <xacro:kinect_gazebo name="kinect_center"/>
   <!-- Kinect_hand -->
   <!-- Link -->
@@ -40,3 +40,37 @@
   <!-- Gazebo -->
   <xacro:kinect_gazebo name="kinect_hand"/>
+  <!-- Kinect_right -->
+  <!-- Link -->
+  <xacro:kinect2_link_box_v0 name="kinect_right_link"/>
+  <link name="kinect_right_rgb_optical_frame"/>
+  <!-- Joint -->
+  <joint name="joint_kinect_right" type="fixed">
+  <origin xyz="-0.5255 -0.9966 0.7635" rpy="-0.0233 0.5223 0.481" />
+    <parent link="base_link"/>
+    <child link="kinect_right_link"/>
+  </joint>
+  <joint name="joint_rgb_kinect_right" type="fixed">
+    <origin rpy="${M_PI/2} ${M_PI} ${M_PI/2}"/>
+    <parent link="kinect_right_link"/>
+    <child link="kinect_right_rgb_optical_frame"/>
+  </joint>
+  <!-- Gazebo -->
+  <xacro:kinect_gazebo name="kinect_right"/>
+  <!-- Kinect_left -->
+  <!-- Link -->
+  <xacro:kinect2_link_box_v0 name="kinect_left_link"/>
+  <link name="kinect_left_rgb_optical_frame"/>
+  <!-- Joint -->
+  <joint name="joint_left_right" type="fixed">
+  <origin xyz="-0.496 1.0085 0.756" rpy="0.0126 0.2924 -0.6483" />
+    <parent link="base_link"/>
+    <child link="kinect_left_link"/>
+  </joint>
+  <joint name="joint_rgb_kinect_left" type="fixed">
+    <origin rpy="${M_PI/2} ${M_PI} ${M_PI/2}"/>
+    <parent link="kinect_left_link"/>
+    <child link="kinect_left_rgb_optical_frame"/>
+  </joint>
+  <!-- Gazebo -->
+  <xacro:kinect_gazebo name="kinect_left"/>
 </robot>

Commit message: [fixed]

File: motoman_description/robots/sia5/sia5_with_dhand_and_multi_kinect.urdf.xacro (robot description, xacro)
@@ -63,5 +63,8 @@
   <!-- Joint -->
   <joint name="joint_left_right" type="fixed">
-  <origin xyz="-0.496 1.0085 0.756" rpy="0.0126 0.2924 -0.6483" />
+  <origin xyz="-0.513 1.0085 0.756" rpy="0.0126 0.2924 -0.634" /> <!-- Calibrated position -->
+  <!--  -->
+  <!-- <origin xyz="-0.600 0.800 0.600" rpy="-0.01 0.3206 -0.4815" /> -->
+  <!-- <origin xyz="-0.500 0.800 0.600" rpy="-0.01 0.3206 -0.4815" /> -->
     <parent link="base_link"/>
     <child link="kinect_left_link"/>

Commit message: [modify] chenge sensor position

File: motoman_description/robots/sia5/sia5_with_dhand_and_multi_kinect.urdf.xacro (robot description, xacro)
@@ -63,8 +63,10 @@
   <!-- Joint -->
   <joint name="joint_left_right" type="fixed">
-  <origin xyz="-0.513 1.0085 0.756" rpy="0.0126 0.2924 -0.634" /> <!-- Calibrated position -->
-  <!--  -->
+  <!-- Calibrated position -->
+  <!-- <origin xyz="-0.513 1.0085 0.756" rpy="0.0126 0.2924 -0.634" /> -->
+  <!-- Test positions -->
   <!-- <origin xyz="-0.600 0.800 0.600" rpy="-0.01 0.3206 -0.4815" /> -->
   <!-- <origin xyz="-0.500 0.800 0.600" rpy="-0.01 0.3206 -0.4815" /> -->
+  <origin xyz="-0.4835 1.0027 0.7524" rpy="0.0126 0.2424 -0.6279" />
     <parent link="base_link"/>
     <child link="kinect_left_link"/>

Commit message: [add] recent changes

File: motoman_description/robots/sia5/sia5_with_dhand_and_multi_kinect.urdf.xacro (robot description, xacro)
@@ -68,5 +68,6 @@
   <!-- <origin xyz="-0.600 0.800 0.600" rpy="-0.01 0.3206 -0.4815" /> -->
   <!-- <origin xyz="-0.500 0.800 0.600" rpy="-0.01 0.3206 -0.4815" /> -->
-  <origin xyz="-0.4835 1.0027 0.7524" rpy="0.0126 0.2424 -0.6279" />
+  <!-- <origin xyz="-0.4835 1.0027 0.7524" rpy="0.0126 0.2424 -0.6279" /> --> <!-- test state -->
+  <origin xyz="-0.485969 1.00226 0.71287" rpy="3.13765 2.87986 2.4732" /><!-- estimated state -->
     <parent link="base_link"/>
     <child link="kinect_left_link"/>
