Commit message: [modify] rename 'kinect_second' to 'kinect_center'

File: motoman_description/robots/sia5/sia5_with_dhand_and_4_kinects.urdf.xacro (robot description, xacro)
@@ -6,21 +6,21 @@
   <xacro:include filename="$(find motoman_description)/robots/sia5/sia5_with_dhand.urdf.xacro"/>
   <!-- add Kinect V2 -->
-  <!-- Kinect_second -->
+  <!-- kinect_center -->
   <!-- Link -->
-  <xacro:kinect2_link_box_v0 name="kinect_second_link"/>
-  <link name="kinect_second_rgb_optical_frame"/>
+  <xacro:kinect2_link_box_v0 name="kinect_center_link"/>
+  <link name="kinect_center_rgb_optical_frame"/>
   <!-- Joint -->
-  <joint name="joint_kinect_second" type="fixed">
+  <joint name="joint_kinect_center" type="fixed">
 	<origin xyz="1.4828 0.0827 0.3932" rpy="-0.0031 0.4431 3.14" />
     <parent link="base_link"/>
-    <child link="kinect_second_link"/>
+    <child link="kinect_center_link"/>
   </joint>
-  <joint name="joint_rgb_kinect_second" type="fixed">
+  <joint name="joint_rgb_kinect_center" type="fixed">
     <origin rpy="${M_PI/2} ${M_PI} ${M_PI/2}"/>
-    <parent link="kinect_second_link"/>
-    <child link="kinect_second_rgb_optical_frame"/>
+    <parent link="kinect_center_link"/>
+    <child link="kinect_center_rgb_optical_frame"/>
   </joint>
   <!-- Gazebo -->
-  <xacro:kinect_gazebo name="kinect_second"/>
+  <xacro:kinect_gazebo name="kinect_center"/>
   <!-- Kinect_hand -->
   <!-- Link -->

Commit message: [modify] kinect center calibration

File: motoman_description/robots/sia5/sia5_with_dhand_and_4_kinects.urdf.xacro (robot description, xacro)
@@ -12,5 +12,5 @@
   <!-- Joint -->
   <joint name="joint_kinect_center" type="fixed">
-	<origin xyz="1.4828 0.0827 0.3932" rpy="-0.0031 0.4431 3.14" />
+    <origin xyz="1.4873 0.0804 0.4047" rpy="-0.0031 0.4321 3.14" />
     <parent link="base_link"/>
     <child link="kinect_center_link"/>

Commit message: [modify] calibrated kinect_center

File: motoman_description/robots/sia5/sia5_with_dhand_and_4_kinects.urdf.xacro (robot description, xacro)
@@ -12,5 +12,6 @@
   <!-- Joint -->
   <joint name="joint_kinect_center" type="fixed">
-    <origin xyz="1.4873 0.0804 0.4047" rpy="-0.0031 0.4321 3.14" />
+    <!-- <origin xyz="1.4784 0.0693 0.4383" rpy="-0.0031 0.4319 3.14" /> -->
+    <origin xyz="1.4784 0.0693 0.4358" rpy="0.046 0.4315 -3.1227"/>
     <parent link="base_link"/>
     <child link="kinect_center_link"/>
