Commit message: [Fix] xacro format to kinetic one

File: motoman_description/robots/sia5/sia5_basic.urdf.xacro (robot description, xacro)
@@ -8,15 +8,15 @@
   <xacro:include filename="$(find motoman_description)/urdf/sia5/body.gazebo.xacro"/>
   <!-- Mass -->
-  <property name="sum_mass" value="30.0" />
+  <xacro:property name="sum_mass" value="30.0" />
   <!-- about mass rate -->
-  <property name="table_mass" value="40.0" />
-  <property name="base_rate" value="8.5" />
-  <property name="s_rate" value="7.7" />
-  <property name="l_rate" value="7.0" />
-  <property name="e_rate" value="1.2" />
-  <property name="u_rate" value="1.0" />
-  <property name="r_rate" value="0.9" />
-  <property name="b_rate" value="0.8" />
-  <property name="t_rate" value="0.5" />
+  <xacro:property name="table_mass" value="40.0" />
+  <xacro:property name="base_rate" value="8.5" />
+  <xacro:property name="s_rate" value="7.7" />
+  <xacro:property name="l_rate" value="7.0" />
+  <xacro:property name="e_rate" value="1.2" />
+  <xacro:property name="u_rate" value="1.0" />
+  <xacro:property name="r_rate" value="0.9" />
+  <xacro:property name="b_rate" value="0.8" />
+  <xacro:property name="t_rate" value="0.5" />
   <!-- Hard ware limits -->
   <!-- Range limits -->
@@ -47,5 +47,5 @@
     <link name="world"/>
     <joint name="world" type="fixed">
-      <insert_block name="origin"/>
+      <xacro:insert_block name="origin"/>
       <parent link="world"/>
       <child link="base_link"/>

File: motoman_description/urdf/common.xacro (robot description, xacro)
@@ -1,4 +1,4 @@
 <?xml version="1.0"?>
-<robot>
-  <property name="M_PI" value="3.14159274"/>
+<robot xmlns:xacro="http://ros.org/wiki/xacro">
+    <xacro:property name="M_PI" value="3.14159274" />
 </robot>

File: motoman_description/urdf/sia5/body.urdf.xacro (robot description, xacro)
@@ -1,5 +1,5 @@
 <?xml version="1.0"?>
 <robot xmlns:xacro="http://ros.org/wiki/xacro">
-  <property name="sum_rate" value="${base_rate + s_rate
+  <xacro:property name="sum_rate" value="${base_rate + s_rate
                                       + l_rate + e_rate
                                       + u_rate + r_rate
