Commit message: [modify] change for demo

File: motoman_description/robots/sia5/sia5_with_dhand_and_3_kinects.urdf.xacro (robot description, xacro)
@@ -12,6 +12,6 @@
   <!-- Joint -->
   <joint name="joint_kinect_center" type="fixed">
-    <!-- <origin xyz="1.4784 0.0693 0.4383" rpy="-0.0031 0.4319 3.14" /> -->
-    <origin xyz="1.4784 0.0693 0.4358" rpy="0.046 0.4315 -3.1227"/>
+    <!-- <origin xyz="1.4784 0.0693 0.4358" rpy="0.046 0.4315 -3.1227"/> -->
+    <origin xyz="1.4505 0.1127 0.4244" rpy="0.0453 0.3982 -3.123"/>
     <parent link="base_link"/>
     <child link="kinect_center_link"/>

Commit message: [modify] calibrated kinect_center

File: motoman_description/robots/sia5/sia5_with_dhand_and_3_kinects.urdf.xacro (robot description, xacro)
@@ -13,5 +13,5 @@
   <joint name="joint_kinect_center" type="fixed">
     <!-- <origin xyz="1.4784 0.0693 0.4358" rpy="0.046 0.4315 -3.1227"/> -->
-    <origin xyz="1.4505 0.1127 0.4244" rpy="0.0453 0.3982 -3.123"/>
+    <origin xyz="1.4305 0.1227 0.4244" rpy="0.0453 0.3982 -3.123"/>
     <parent link="base_link"/>
     <child link="kinect_center_link"/>
